Commit message: heavy cfg

File: resources/robots/j60/urdf/z2_heavy.urdf (robot description, URDF)
Before this commit: robot robot, 18 links, 17 joints
Links:
- link FL_calf: mass 0.153 -> 0.175
- link FL_hip: mass 0.614 -> 0.706
- link FL_thigh: mass 1.057 -> 1.215
- link FR_calf: mass 0.153 -> 0.175
- link FR_hip: mass 0.614 -> 0.706
- link FR_thigh: mass 1.057 -> 1.215
- link RL_calf: mass 0.153 -> 0.175
- link RL_hip: mass 0.614 -> 0.706
- link RL_thigh: mass 1.057 -> 1.215
- link RR_calf: mass 0.153 -> 0.175
- link RR_hip: mass 0.614 -> 0.706
- link RR_thigh: mass 1.057 -> 1.215
- link base: mass 3.728 -> 4.287
- link base_imu: mass 0.01 -> 0.51

Commit message: him ready for test

File: resources/robots/j60/urdf/z2_heavy.urdf (robot description, URDF)
Before this commit: robot robot, 18 links, 17 joints
Joints:
- joint FL_hip_joint: limit lower=--0.5 upper=-0.5 effort=30 velocity=15 -> lower=-0.5 upper=0.5 effort=30 velocity=15
- joint FR_hip_joint: limit lower=--0.5 upper=-0.5 effort=30 velocity=15 -> lower=-0.5 upper=0.5 effort=30 velocity=15
- joint RL_hip_joint: limit lower=--0.5 upper=-0.5 effort=30 velocity=15 -> lower=-0.5 upper=0.5 effort=30 velocity=15
- joint RR_hip_joint: limit lower=--0.5 upper=-0.5 effort=30 velocity=15 -> lower=-0.5 upper=0.5 effort=30 velocity=15
