Commit message: new z2 fixed

File: resources/robots/aaaaa_fixed/z2/urdf/z2.urdf (robot description, URDF)
Before this commit: robot z2, 17 links, 16 joints
Links:
- link FL_calf: geometry collision box size=0.2403 0.04 0.03; visual mesh filename=../meshes/FL_calf.STL
- link FL_foot: geometry collision sphere radius=0.026; visual mesh filename=../meshes/FL_foot.STL
- link FL_hip: geometry collision cylinder length=0.0668 radius=0.0366; visual mesh filename=../meshes/FL_hip.STL
- link FL_thigh: geometry collision box size=0.05 0.03 0.19; collision cylinder length=0.1005 radius=0.0422
- link FR_calf: geometry collision box size=0.2403 0.04 0.03; visual mesh filename=../meshes/FR_calf.STL
- link FR_foot: geometry collision sphere radius=0.026; visual mesh filename=../meshes/FR_foot.STL
- link FR_hip: geometry collision cylinder length=0.0668 radius=0.0366; visual mesh filename=../meshes/FR_hip.STL
- link FR_thigh: geometry collision box size=0.05 0.03 0.19; collision cylinder length=0.1005 radius=0.0422
- link RL_calf: geometry collision box size=0.2403 0.04 0.03; visual mesh filename=../meshes/RL_calf.STL
- link RL_foot: geometry collision sphere radius=0.026; visual mesh filename=../meshes/RL_foot.STL
- link RL_hip: geometry collision cylinder length=0.0668 radius=0.0366; visual mesh filename=../meshes/RL_hip.STL
- link RL_thigh: geometry collision box size=0.05 0.03 0.19; collision cylinder length=0.1005 radius=0.0422
- link RR_calf: geometry collision box size=0.2403 0.04 0.03; visual mesh filename=../meshes/RR_calf.STL
- link RR_foot: geometry collision sphere radius=0.026; visual mesh filename=../meshes/RR_foot.STL
- link RR_hip: geometry collision cylinder length=0.0668 radius=0.0366; visual mesh filename=../meshes/RR_hip.STL
- link RR_thigh: geometry collision box size=0.05 0.03 0.19; collision cylinder length=0.1005 radius=0.0422
- link base_link: geometry collision box size=0.342 0.2369992 0.0869992; visual mesh filename=../meshes/base_link.STL

Commit message: j60 urdf

File: resources/robots/aaaaa_fixed/z2/urdf/z2.urdf (robot description, URDF)
Before this commit: robot z2, 17 links, 16 joints
Joints:
- joint FL_calf_joint: limit lower=-2.4 upper=-0.3 effort=30 velocity=15 -> lower=-2.4 upper=-1.1 effort=30 velocity=15
- joint FL_thigh_joint: limit lower=-0.3 upper=3.2 effort=30 velocity=15 -> lower=-0.1 upper=3.2 effort=30 velocity=15
- joint FR_calf_joint: limit lower=-2.4 upper=-0.3 effort=30 velocity=15 -> lower=-2.4 upper=-1.1 effort=30 velocity=15
- joint FR_thigh_joint: limit lower=-0.3 upper=3.2 effort=30 velocity=15 -> lower=-0.1 upper=3.2 effort=30 velocity=15
- joint RL_calf_joint: limit lower=-2.4 upper=-0.3 effort=30 velocity=15 -> lower=-2.4 upper=-1.1 effort=30 velocity=15
- joint RL_thigh_joint: limit lower=-0.3 upper=3.2 effort=30 velocity=15 -> lower=-0.1 upper=3.2 effort=30 velocity=15
- joint RR_calf_joint: limit lower=-2.4 upper=-0.3 effort=30 velocity=15 -> lower=-2.4 upper=-1.1 effort=30 velocity=15
- joint RR_thigh_joint: limit lower=-0.3 upper=3.2 effort=30 velocity=15 -> lower=-0.1 upper=3.2 effort=30 velocity=15

File: resources/robots/j60/urdf/z2_heavy.urdf (robot description, URDF)
Before this commit: robot robot, 18 links, 17 joints
Joints:
- joint FL_hip_joint: limit lower=-0.8028514559173915 upper=0.8028514559173915 effort=30 velocity=15 -> lower=--0.5 upper=-0.5 effort=30 velocity=15
- joint FL_thigh_joint: limit lower=-1.0471975511965976 upper=4.1887902047863905 effort=30 velocity=15 -> lower=-0.10 upper=3.10 effort=30 velocity=15
- joint FR_hip_joint: limit lower=-0.8028514559173915 upper=0.8028514559173915 effort=30 velocity=15 -> lower=--0.5 upper=-0.5 effort=30 velocity=15
- joint FR_thigh_joint: limit lower=-1.0471975511965976 upper=4.1887902047863905 effort=30 velocity=15 -> lower=-0.10 upper=3.10 effort=30 velocity=15
- joint RL_hip_joint: limit lower=-0.8028514559173915 upper=0.8028514559173915 effort=30 velocity=15 -> lower=--0.5 upper=-0.5 effort=30 velocity=15
- joint RL_thigh_joint: limit lower=-1.0471975511965976 upper=4.1887902047863905 effort=30 velocity=15 -> lower=-0.10 upper=3.10 effort=30 velocity=15
- joint RR_hip_joint: limit lower=-0.8028514559173915 upper=0.8028514559173915 effort=30 velocity=15 -> lower=--0.5 upper=-0.5 effort=30 velocity=15
- joint RR_thigh_joint: limit lower=-1.0471975511965976 upper=4.1887902047863905 effort=30 velocity=15 -> lower=-0.10 upper=3.10 effort=30 velocity=15

Commit message: urdf微调

File: resources/robots/aaaaa_fixed/z2/urdf/z2.urdf (robot description, URDF)
Before this commit: robot z2, 17 links, 16 joints
Joints:
- joint FL_calf_joint: limit lower=-2.4 upper=-1.1 effort=30 velocity=15 -> lower=-2.6965337 upper=-0.9162979 effort=30 velocity=15
- joint FL_foot_joint: origin xyz=0.0450727 0.0002 -0.205232 rpy=0 0 0 -> xyz=0 0.0002 -0.21012 rpy=0 0 0
- joint FR_calf_joint: limit lower=-2.4 upper=-1.1 effort=30 velocity=15 -> lower=-2.6965337 upper=-0.9162979 effort=30 velocity=15
- joint FR_foot_joint: origin xyz=0.0499776 -0.0002 -0.204093 rpy=0 0 0 -> xyz=0 -0.0002 -0.21012 rpy=0 0 0
- joint RL_calf_joint: limit lower=-2.4 upper=-1.1 effort=30 velocity=15 -> lower=-2.6965337 upper=-0.9162979 effort=30 velocity=15
- joint RL_foot_joint: origin xyz=0.0450727 0.0002 -0.205232 rpy=0 0 0 -> xyz=0 0.0002 -0.2101231 rpy=0 0 0
- joint RR_calf_joint: limit lower=-2.4 upper=-1.1 effort=30 velocity=15 -> lower=-2.6965337 upper=-0.9162979 effort=30 velocity=15
- joint RR_foot_joint: origin xyz=0.0499776 -0.0002 -0.204093 rpy=0 0 0 -> xyz=0 -0.0002 -0.21012 rpy=0 0 0
