Commit message: Update z2.urdf

File: resources/robots/aaaaa_fixed/z2/urdf/z2.urdf (robot description, URDF)
Before this commit: robot z2, 17 links, 16 joints
Links:
- link FL_calf: mass 0.18 -> 0.1421
- link FL_foot: mass 0.02 -> 0.0241
- link FL_thigh: mass 0.955 -> 1.013
- link FR_calf: mass 0.18 -> 0.1421
- link FR_foot: mass 0.02 -> 0.0241
- link FR_thigh: mass 0.955 -> 1.013
- link RL_calf: mass 0.18 -> 0.1421
- link RL_foot: mass 0.02 -> 0.0241
- link RL_thigh: mass 0.955 -> 1.013
- link RR_calf: mass 0.18 -> 0.1421
- link RR_foot: mass 0.02 -> 0.0241
- link RR_thigh: mass 0.955 -> 1.013
- link base_link: mass 5.58 -> 6.32
